File: kicad/axoloti_429_eurorack/pots_cv_inputs.sch (KiCad schematic (older format))
At the start: 86 parts, among them J20 JACK_CV_IN1, J21 JACK_CV_IN2, J22 JACK_CV_IN3, J23 JACK_CV_IN4, J24 JACK_CV_IN5, J25 JACK_CV_IN6, J26 JACK_CV_IN7, J27 JACK_CV_IN8, U14 MCP6004, U15 MCP6004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

Commit message: boot, reset switches
Parts:
- R69, R75, R79, R83, R87, R91, R95, R99: value 30k -> 33k
Connections:
- net AREF_3V0 renamed AREF_3V3
Changed lines of the file:
@@
 $EndComp
 Text GLabel 3350 1300 0    50   Input ~ 0
-AREF_3V0
+AREF_3V3
 Wire Wire Line
 	3350 1300 3350 1375
@@
 AR Path="/61EC8332/61EE0BFD" Ref="R69"  Part="1"
 F 0 "R69" V 3600 1525 50  0000 C CNN
-F 1 "30k" V 3700 1525 50  0000 C CNN
+F 1 "33k" V 3700 1525 50  0000 C CNN
 F 2 "" V 3630 1525 50  0001 C CNN
 F 3 "~" H 3700 1525 50  0001 C CNN
@@
 $EndComp
 Text GLabel 8250 1200 0    50   Input ~ 0
-AREF_3V0
+AREF_3V3
 Wire Wire Line
 	8250 1200 8250 1275
@@
 AR Path="/61EC8332/61EEBE5B" Ref="R75"  Part="1"
 F 0 "R75" V 8500 1425 50  0000 C CNN
-F 1 "30k" V 8600 1425 50  0000 C CNN
+F 1 "33k" V 8600 1425 50  0000 C CNN
 F 2 "" V 8530 1425 50  0001 C CNN
 F 3 "~" H 8600 1425 50  0001 C CNN
@@
 $EndComp
 Text GLabel 3225 3350 0    50   Input ~ 0
-AREF_3V0
+AREF_3V3
 Wire Wire Line
 	3225 3350 3225 3425
@@
 AR Path="/61EC8332/61EF0320" Ref="R79"  Part="1"
 F 0 "R79" V 3475 3575 50  0000 C CNN
-F 1 "30k" V 3575 3575 50  0000 C CNN
+F 1 "33k" V 3575 3575 50  0000 C CNN
 F 2 "" V 3505 3575 50  0001 C CNN
 F 3 "~" H 3575 3575 50  0001 C CNN
@@
 $EndComp
 Text GLabel 8175 3250 0    50   Input ~ 0
-AREF_3V0
+AREF_3V3
 Wire Wire Line
 	8175 3250 8175 3325
@@
 AR Path="/61EC8332/61EF4954" Ref="R83"  Part="1"
 F 0 "R83" V 8425 3475 50  0000 C CNN
-F 1 "30k" V 8525 3475 50  0000 C CNN
+F 1 "33k" V 8525 3475 50  0000 C CNN
 F 2 "" V 8455 3475 50  0001 C CNN
 F 3 "~" H 8525 3475 50  0001 C CNN
@@
 $EndComp
 Text GLabel 1400 5325 0    50   Input ~ 0
-AREF_3V0
+AREF_3V3
 Wire Wire Line
 	1400 5325 1400 5400
@@
 AR Path="/61EC8332/621E97EF" Ref="R87"  Part="1"
 F 0 "R87" V 1650 5550 50  0000 C CNN
-F 1 "30k" V 1750 5550 50  0000 C CNN
+F 1 "33k" V 1750 5550 50  0000 C CNN
 F 2 "" V 1680 5550 50  0001 C CNN
 F 3 "~" H 1750 5550 50  0001 C CNN
@@
 $EndComp
 Text GLabel 3925 5300 0    50   Input ~ 0
-AREF_3V0
+AREF_3V3
 Wire Wire Line
 	3925 5300 3925 5375
@@
 AR Path="/61EC8332/621E9855" Ref="R91"  Part="1"
 F 0 "R91" V 4175 5525 50  0000 C CNN
-F 1 "30k" V 4275 5525 50  0000 C CNN
+F 1 "33k" V 4275 5525 50  0000 C CNN
 F 2 "" V 4205 5525 50  0001 C CNN
 F 3 "~" H 4275 5525 50  0001 C CNN
@@
 $EndComp
 Text GLabel 6475 5325 0    50   Input ~ 0
-AREF_3V0
+AREF_3V3
 Wire Wire Line
 	6475 5325 6475 5400
@@
 AR Path="/61EC8332/621E98B5" Ref="R95"  Part="1"
 F 0 "R95" V 6725 5550 50  0000 C CNN
-F 1 "30k" V 6825 5550 50  0000 C CNN
+F 1 "33k" V 6825 5550 50  0000 C CNN
 F 2 "" V 6755 5550 50  0001 C CNN
 F 3 "~" H 6825 5550 50  0001 C CNN
@@
 $EndComp
 Text GLabel 9100 5350 0    50   Input ~ 0
-AREF_3V0
+AREF_3V3
 Wire Wire Line
 	9100 5350 9100 5425
@@
 AR Path="/61EC8332/621E9915" Ref="R99"  Part="1"
 F 0 "R99" V 9350 5575 50  0000 C CNN
-F 1 "30k" V 9450 5575 50  0000 C CNN
+F 1 "33k" V 9450 5575 50  0000 C CNN
 F 2 "" V 9380 5575 50  0001 C CNN
 F 3 "~" H 9450 5575 50  0001 C CNN
