File: kicad/axoloti_429_eurorack/axoloti_429_eurorack.sch (KiCad schematic (older format))
At the start: 40 parts, among them J1 SERIAL_SYSTEM_BOOTLOADER, J11 I2C1_HEADER, J30 429_Conn_02x27_Odd_Even_mirro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, J8 429_Conn_02x27_Odd_Even, SW1 BOOT_FLASH, SW2 RESET, U2 STM32F427IITx, Y1 8Mhz

Commit message: boot, reset switches
Parts:
- removed C33, C34: 2.2u, symbol Device:C_Small
- removed C35, C67: 1u, symbol Device:C_Small
- removed C36: 10n, symbol Device:C_Small
- removed C37, C38, C46, C47, C48, C50, C51, C52, C53, C55, C56, C57, C58, C68, C69, C70: 100n, symbol Device:C_Small
- removed C49: 4.7u, symbol Device:CP_Small
- removed C54: C_Small, symbol Device:C_Small
- removed C59, C60: 18p, symbol Device:C_Small
- removed R36, R41: 10k, Resistor_SMD:R_0603_1608Metric, symbol Device:R
- removed SW2: RESET, Button_Switch_SMD:SW_Push_1P1T_NO_6x6mm_H9.5mm, symbol Switch:SW_MEC_5E
- removed Y1: 8Mhz, Crystal:Crystal_HC49-U_Vertical, symbol Device:Crystal
Connections:
- net +3V3: no longer U2.103 (VDD), U2.114 (VDD), U2.127 (VDD), U2.136 (VDD), U2.149 (VDD), U2.15 (VDD), U2.159 (VDD), U2.171 (PDR_ON), U2.172 (VDD), U2.23 (VDD), U2.36 (VDD), U2.49 (VDD), U2.6 (VBAT), U2.62 (VDD), U2.72 (VDD), U2.82 (VDD), U2.91 (VDD)
- net 2141_EN: now also J8.13 (PD7); no longer U2.151 (FMC_NCE2/FMC_NE1/USART2_CK/PD7)
- net 2141_FLG: now also J8.20 (PG13); no longer U2.156 (PG13/ETH_TXD0/FMC_A24/SPI6_SCK/USART6_CTS)
- net BOOT_FLASH: now also J8.28 (BOOT0); no longer U2.166 (BOOT0)
- net CV_IN1: now also J8.49 (PA0); no longer U2.40 (ADC1_IN0/ADC2_IN0/ADC3_IN0/ETH_CRS/SYS_WKUP/TIM2_CH1/TIM2_ETR/TIM5_CH1/TIM8_ETR/UART4_TX/USART2_CTS/PA0)
- net CV_IN2: now also J8.52 (PA1); no longer U2.41 (ADC1_IN1/ADC2_IN1/ADC3_IN1/ETH_REF_CLK/ETH_RX_CLK/TIM2_CH2/TIM5_CH2/UART4_RX/USART2_RTS/PA1)
- net CV_IN3: now also J8.51 (PA2); no longer U2.42 (ADC1_IN2/ADC2_IN2/ADC3_IN2/ETH_MDIO/TIM2_CH3/TIM5_CH3/TIM9_CH1/USART2_TX/PA2)
- net CV_IN4: now also J30.43 (PA3); no longer U2.47 (ADC1_IN3/ADC2_IN3/ADC3_IN3/ETH_COL/TIM2_CH4/TIM5_CH4/TIM9_CH2/USART2_RX/USB_OTG_HS_ULPI_D0/PA3)
- net DAC_OUT1: now also J30.44 (PA4); no longer U2.50 (ADC1_IN4/ADC2_IN4/DAC_OUT1/DCMI_HSYNC/I2S3_WS/SPI1_NSS/SPI3_NSS/USART2_CK/USB_OTG_HS_SOF/PA4)
- net DAC_OUT2: now also J30.41 (PA5); no longer U2.51 (ADC1_IN5/ADC2_IN5/DAC_OUT2/SPI1_SCK/TIM2_CH1/TIM2_ETR/TIM8_CH1N/USB_OTG_HS_ULPI_CK/PA5)
- net GND: no longer U2.102 (VSS), U2.113 (VSS), U2.126 (VSS), U2.135 (VSS), U2.14 (VSS), U2.148 (VSS), U2.158 (VSS), U2.22 (VSS), U2.48 (BYPASS_REG), U2.61 (VSS), U2.71 (VSS), U2.90 (VSS)
- net LED_GREEN: now also J30.20 (PG6); no longer U2.110 (PG6/DCMI_D12/FMC_INT2)
- net LED_RED: now also J30.18 (PC6); no longer U2.115 (DCMI_D0/I2S2_MCK/SDIO_D6/TIM3_CH1/TIM8_CH1/USART6_TX/PC6)
- net MIDI_RX: now also J8.16 (PG9); no longer U2.152 (PG9/DAC_EXTI9/DCMI_VSYNC/FMC_NCE3/FMC_NE2/USART6_RX)
- net MIDI_TX: now also J8.19 (PG14); no longer U2.157 (PG14/ETH_TXD1/FMC_A25/SPI6_MOSI/USART6_TX)
- net SAI1_FS_A: now also J8.35 (PE4); no longer U2.3 (DCMI_D4/FMC_A20/SAI1_FS_A/SPI4_NSS/SYS_TRACED1/PE4)
- net SAI1_SCK_A: now also J8.38 (PE5); no longer U2.4 (DCMI_D6/FMC_A21/SAI1_SCK_A/SPI4_MISO/SYS_TRACED2/TIM9_CH1/PE5)
- net SAI1_SD_A: now also J8.37 (PE6); no longer U2.5 (DCMI_D7/FMC_A22/SAI1_SD_A/SPI4_MOSI/SYS_TRACED3/TIM9_CH2/PE6)
- net SAI1_SD_B: now also J8.36 (PE3); no longer U2.2 (FMC_A19/SAI1_SD_B/SYS_TRACED0/PE3)
- net V_SUPERVIS: now also J8.43 (PF10); no longer U2.28 (PF10/ADC3_IN8/DCMI_D11/FMC_INTR)
- net +3.3VA: no longer names the net of U2.39 (VDDA)
- net AREF_3V0: no longer names the net of U2.38 (VREF+)
- net FMC_A0: no longer names the net of U2.16 (PF0/FMC_A0/I2C2_SDA)
- net FMC_A1: no longer names the net of U2.17 (PF1/FMC_A1/I2C2_SCL)
- net FMC_A10: no longer names the net of U2.66 (PG0/FMC_A10)
- net FMC_A11: no longer names the net of U2.67 (PG1/FMC_A11)
- net FMC_A12: no longer names the net of U2.106 (PG2/FMC_A12)
- net FMC_A2: no longer names the net of U2.18 (PF2/FMC_A2/I2C2_SMBA)
- net FMC_A3: no longer names the net of U2.19 (PF3/ADC3_IN9/FMC_A3)
- net FMC_A4: no longer names the net of U2.20 (PF4/ADC3_IN14/FMC_A4)
- net FMC_A5: no longer names the net of U2.21 (PF5/ADC3_IN15/FMC_A5)
- net FMC_A6: no longer names the net of U2.60 (PF12/FMC_A6)
- net FMC_A7: no longer names the net of U2.63 (PF13/FMC_A7)
- net FMC_A8: no longer names the net of U2.64 (PF14/FMC_A8)
- net FMC_A9: no longer names the net of U2.65 (PF15/ADC1_EXTI15/ADC2_EXTI15/ADC3_EXTI15/FMC_A9)
- net FMC_BA0: no longer names the net of U2.108 (PG4/FMC_A14/FMC_BA0)
- net FMC_BA1: no longer names the net of U2.109 (PG5/FMC_A15/FMC_BA1)
- net FMC_CAS: no longer names the net of U2.160 (PG15/ADC1_EXTI15/ADC2_EXTI15/ADC3_EXTI15/DCMI_D13/FMC_SDNCAS/USART6_CTS)
- net FMC_D0: no longer names the net of U2.104 (FMC_D0/FMC_DA0/TIM4_CH3/PD14)
- net FMC_D1: no longer names the net of U2.105 (ADC1_EXTI15/ADC2_EXTI15/ADC3_EXTI15/FMC_D1/FMC_DA1/TIM4_CH4/PD15)
- net FMC_D10: no longer names the net of U2.76 (FMC_D10/FMC_DA10/SPI4_MISO/TIM1_CH3/PE13)
- net FMC_D11: no longer names the net of U2.77 (FMC_D11/FMC_DA11/SPI4_MOSI/TIM1_CH4/PE14)
- net FMC_D12: no longer names the net of U2.78 (ADC1_EXTI15/ADC2_EXTI15/ADC3_EXTI15/FMC_D12/FMC_DA12/TIM1_BKIN/PE15)
- net FMC_D13: no longer names the net of U2.96 (FMC_D13/FMC_DA13/USART3_TX/PD8)
- net FMC_D14: no longer names the net of U2.97 (DAC_EXTI9/FMC_D14/FMC_DA14/USART3_RX/PD9)
- net FMC_D15: no longer names the net of U2.98 (FMC_D15/FMC_DA15/USART3_CK/PD10)
- net FMC_D2: no longer names the net of U2.142 (CAN1_RX/FMC_D2/FMC_DA2/PD0)
- net FMC_D3: no longer names the net of U2.143 (CAN1_TX/FMC_D3/FMC_DA3/PD1)
- net FMC_D4: no longer names the net of U2.68 (FMC_D4/FMC_DA4/TIM1_ETR/UART7_RX/PE7)
- net FMC_D5: no longer names the net of U2.69 (FMC_D5/FMC_DA5/TIM1_CH1N/UART7_TX/PE8)
- net FMC_D6: no longer names the net of U2.70 (DAC_EXTI9/FMC_D6/FMC_DA6/TIM1_CH1/PE9)
- net FMC_D7: no longer names the net of U2.73 (FMC_D7/FMC_DA7/TIM1_CH2N/PE10)
- net FMC_D8: no longer names the net of U2.74 (ADC1_EXTI11/ADC2_EXTI11/ADC3_EXTI11/FMC_D8/FMC_DA8/SPI4_NSS/TIM1_CH2/PE11)
- net FMC_D9: no longer names the net of U2.75 (FMC_D9/FMC_DA9/SPI4_SCK/TIM1_CH3N/PE12)
- net FMC_NBL0: no longer names the net of U2.169 (DCMI_D2/FMC_NBL0/TIM4_ETR/UART8_RX/PE0)
- net FMC_NBL1: no longer names the net of U2.170 (DCMI_D3/FMC_NBL1/UART8_TX/PE1)
- net FMC_RAS: no longer names the net of U2.59 (PF11/ADC1_EXTI11/ADC2_EXTI11/ADC3_EXTI11/DCMI_D12/FMC_SDNRAS/SPI5_MOSI)
- net FMC_SDCKE0: no longer names the net of U2.43 (PH2/ETH_CRS/FMC_SDCKE0)
- net FMC_SDCKE1: no longer names the net of U2.84 (PH7/DCMI_D9/ETH_RXD3/FMC_SDCKE1/I2C3_SCL/SPI5_MISO)
- net FMC_SDCLK: no longer names the net of U2.112 (PG8/ETH_PPS_OUT/FMC_SDCLK/SPI6_NSS/USART6_RTS)
- net FMC_SDNE0: no longer names the net of U2.44 (PH3/ETH_COL/FMC_SDNE0)
- net FMC_SDNE1: no longer names the net of U2.83 (PH6/DCMI_D8/ETH_RXD2/FMC_SDNE1/I2C2_SMBA/SPI5_SCK/TIM12_CH1)
- net FMC_SDNWE: no longer names the net of U2.46 (PH5/FMC_SDNWE/I2C2_SDA/SPI5_NSS)
- net GNDA: no longer names the net of U2.37 (VSSA)
- net RESET: no longer names the net of U2.31 (NRST)
- new net: U2.103 (VDD), U2.114 (VDD), U2.127 (VDD), U2.136 (VDD), U2.149 (VDD), U2.15 (VDD), U2.159 (VDD), U2.172 (VDD), U2.23 (VDD), U2.36 (VDD), U2.49 (VDD), U2.62 (VDD), U2.72 (VDD), U2.82 (VDD), U2.91 (VDD)
- no-connect marks 9 -> 10
Other:
- note added: "LCtech already includes 10k pull down"
- note added: "TODO"
- moved on the sheet: J8

Commit message: create README.md
Other:
- moved on the sheet: J30
Changed lines of the file:
@@
 Wire Wire Line
 	12000 6925 11775 6925
-Text GLabel -2200 11800 0    50   Input ~ 0
+Text GLabel -850 10200 2    50   Input ~ 0
 DAC_OUT1
 Wire Wire Line
-	-2200 11800 -2100 11800
-Text GLabel -700 11700 2    50   Input ~ 0
+	-850 10200 -950 10200
+Text GLabel -2350 10300 0    50   Input ~ 0
 DAC_OUT2
 Wire Wire Line
-	-800 11700 -700 11700
+	-2250 10300 -2350 10300
 Text GLabel 11875 2725 2    50   Input ~ 0
 OTG_FS_DM
@@
 Text GLabel -5325 12200 0    50   Input ~ 0
 CV_IN3
-Text GLabel -675 11800 2    50   Input ~ 0
+Text GLabel -2375 10200 0    50   Input ~ 0
 CV_IN4
 Text GLabel 11900 2225 2    50   Input ~ 0
@@
 	-5325 12200 -5200 12200
 Wire Wire Line
-	-800 11800 -675 11800
+	-2250 10200 -2375 10200
 Wire Wire Line
 	11775 2225 11900 2225
@@
 Text Notes 15325 2400 0    50   ~ 0
 done
-Text GLabel -2400 10500 0    50   Input ~ 0
+Text GLabel -650 11500 2    50   Input ~ 0
 LED_RED
 Wire Wire Line
-	-2400 10500 -2100 10500
-Text GLabel -2350 10600 0    50   Input ~ 0
+	-650 11500 -950 11500
+Text GLabel -700 11400 2    50   Input ~ 0
 LED_GREEN
 Wire Wire Line
-	-2350 10600 -2100 10600
+	-700 11400 -950 11400
 Text GLabel 11875 2425 2    50   Input ~ 0
 SAI_MCLK
@@
 L power:GND #PWR0146
 U 1 1 616899AD
-P -2375 12100
-F 0 "#PWR0146" H -2375 11850 50  0001 C CNN
-F 1 "GND" V -2370 11972 50  0000 R CNN
-F 2 "" H -2375 12100 50  0001 C CNN
-F 3 "" H -2375 12100 50  0001 C CNN
-	1    -2375 12100
-	0    1    1    0
-$EndComp
-Wire Wire Line
-	-2375 12100 -2100 12100
+P -675 9900
+F 0 "#PWR0146" H -675 9650 50  0001 C CNN
+F 1 "GND" V -670 9772 50  0000 R CNN
+F 2 "" H -675 9900 50  0001 C CNN
+F 3 "" H -675 9900 50  0001 C CNN
+	1    -675 9900
+	0    -1   -1   0
+$EndComp
+Wire Wire Line
+	-675 9900 -950 9900
 $Comp
 L power:+3.3V #PWR0147
 U 1 1 616BAD54
-P -2375 12200
-F 0 "#PWR0147" H -2375 12050 50  0001 C CNN
-F 1 "+3.3V" V -2360 12328 50  0000 L CNN
-F 2 "" H -2375 12200 50  0001 C CNN
-F 3 "" H -2375 12200 50  0001 C CNN
-	1    -2375 12200
-	0    -1   -1   0
-$EndComp
-Wire Wire Line
-	-2375 12200 -2100 12200
+P -675 9800
+F 0 "#PWR0147" H -675 9650 50  0001 C CNN
+F 1 "+3.3V" V -660 9928 50  0000 L CNN
+F 2 "" H -675 9800 50  0001 C CNN
+F 3 "" H -675 9800 50  0001 C CNN
+	1    -675 9800
+	0    1    1    0
+$EndComp
+Wire Wire Line
+	-675 9800 -950 9800
 $Comp
 L power:+5V #PWR0148
 U 1 1 616EEC4D
-P -2375 12300
-F 0 "#PWR0148" H -2375 12150 50  0001 C CNN
-F 1 "+5V" V -2360 12428 50  0000 L CNN
-F 2 "" H -2375 12300 50  0001 C CNN
-F 3 "" H -2375 12300 50  0001 C CNN
-	1    -2375 12300
-	0    -1   -1   0
-$EndComp
-Wire Wire Line
-	-2375 12300 -2100 12300
+P -675 9700
+F 0 "#PWR0148" H -675 9550 50  0001 C CNN
+F 1 "+5V" V -660 9828 50  0000 L CNN
+F 2 "" H -675 9700 50  0001 C CNN
+F 3 "" H -675 9700 50  0001 C CNN
+	1    -675 9700
+	0    1    1    0
+$EndComp
+Wire Wire Line
+	-675 9700 -950 9700
 Text GLabel -3625 9800 2    50   Input ~ 0
 VBAT
@@
 Wire Wire Line
 	-5475 11800 -5200 11800
-$Comp
-L w_connector:429_Conn_02x27_Odd_Even_mirrored J30
-U 1 1 617A73CC
-P -1450 11000
-F 0 "J30" H -1450 12517 50  0000 C CNN
-F 1 "429_Conn_02x27_Odd_Even_mirrored" H -1450 12426 50  0000 C CNN
-F 2 "" H -1200 11000 50  0001 C CNN
-F 3 "~" H -1200 11000 50  0001 C CNN
-	1    -1450 11000
-	1    0    0    -1
-$EndComp
 Text GLabel -4375 8375 2    50   Input ~ 0
 V_SUPERVIS
@@
 $EndComp
 Wire Wire Line
-	-525 12300 -800 12300
+	-2525 9700 -2250 9700
 $Comp
 L power:+5V #PWR0152
 U 1 1 61707F5F
-P -525 12300
-F 0 "#PWR0152" H -525 12150 50  0001 C CNN
-F 1 "+5V" V -510 12428 50  0000 L CNN
-F 2 "" H -525 12300 50  0001 C CNN
-F 3 "" H -525 12300 50  0001 C CNN
-	1    -525 12300
-	0    1    1    0
-$EndComp
-Wire Wire Line
-	-525 12200 -800 12200
+P -2525 9700
+F 0 "#PWR0152" H -2525 9550 50  0001 C CNN
+F 1 "+5V" V -2510 9828 50  0000 L CNN
+F 2 "" H -2525 9700 50  0001 C CNN
+F 3 "" H -2525 9700 50  0001 C CNN
+	1    -2525 9700
+	0    -1   -1   0
+$EndComp
+Wire Wire Line
+	-2525 9800 -2250 9800
 $Comp
 L power:+3.3V #PWR0151
 U 1 1 616D3BDC
-P -525 12200
-F 0 "#PWR0151" H -525 12050 50  0001 C CNN
-F 1 "+3.3V" V -510 12328 50  0000 L CNN
-F 2 "" H -525 12200 50  0001 C CNN
-F 3 "" H -525 12200 50  0001 C CNN
-	1    -525 12200
-	0    1    1    0
-$EndComp
-Wire Wire Line
-	-525 12100 -800 12100
+P -2525 9800
+F 0 "#PWR0151" H -2525 9650 50  0001 C CNN
+F 1 "+3.3V" V -2510 9928 50  0000 L CNN
+F 2 "" H -2525 9800 50  0001 C CNN
+F 3 "" H -2525 9800 50  0001 C CNN
+	1    -2525 9800
+	0    -1   -1   0
+$EndComp
+Wire Wire Line
+	-2525 9900 -2250 9900
 $Comp
 L power:GND #PWR0150
 U 1 1 616A1448
-P -525 12100
-F 0 "#PWR0150" H -525 11850 50  0001 C CNN
-F 1 "GND" V -520 11972 50  0000 R CNN
-F 2 "" H -525 12100 50  0001 C CNN
-F 3 "" H -525 12100 50  0001 C CNN
-	1    -525 12100
-	0    -1   -1   0
+P -2525 9900
+F 0 "#PWR0150" H -2525 9650 50  0001 C CNN
+F 1 "GND" V -2520 9772 50  0000 R CNN
+F 2 "" H -2525 9900 50  0001 C CNN
+F 3 "" H -2525 9900 50  0001 C CNN
+	1    -2525 9900
+	0    1    1    0
 $EndComp
 Text GLabel -5450 10600 0    50   Input ~ 0
@@
 LCtech already includes 10k pull down
 NoConn ~ -3900 11900
+$Comp
+L w_connector:429_Conn_02x27_Odd_Even_mirrored J30
+U 1 1 617A73CC
+P -1600 11000
+F 0 "J30" H -1600 12517 50  0000 C CNN
+F 1 "429_Conn_02x27_Odd_Even_mirrored" H -1600 12426 50  0000 C CNN
+F 2 "" H -1350 11000 50  0001 C CNN
+F 3 "~" H -1350 11000 50  0001 C CNN
+	1    -1600 11000
+	-1   0    0    1
+$EndComp
 $EndSCHEMATC

Commit message: cleanup
Parts:
- removed U2: STM32F427IITx, LQFP176, symbol w_stm32:STM32F427IITx
Connections:
- wire segments 126 -> 96
- no-connect marks 10 -> 8
Other:
- note added: "I2C pull-ups"
- note removed: "VCC\nGND"
- note removed: "warning: PC13, 14, 15 are weak"
- moved on the sheet: C83, J1, J11, J30, J8, R105, R106, R21, R23, SW1
