File: kicad/axoloti_429_eurorack/digital_io.sch (KiCad schematic (older format))
At the start: 66 parts, among them J10 JACK_GATE_IN2, J19 JACK_GATE_OUT2, J28 JACK_CV_OUT1, J29 JACK_CV_OUT1, J3 JACK_GATE_OUT1, J9 JACK_GATE_IN1, Q1 MMBT3904, Q2 MMBT3904, U12 TL074, U19 TL072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

Commit message: boot, reset switches
Parts:
- added C33, C34, C35, C36: 100n, symbol Device:C_Small
- added R102, R58: 10k, Resistor_SMD:R_0603_1608Metric, symbol Device:R
- added SW3: BUTTON1, Button_Switch_SMD:SW_Push_1P1T_NO_6x6mm_H9.5mm, symbol Switch:SW_MEC_5E
- added SW4: BUTTON2, Button_Switch_SMD:SW_Push_1P1T_NO_6x6mm_H9.5mm, symbol Switch:SW_MEC_5E
- added SW5: BUTTON3, Button_Switch_SMD:SW_Push_1P1T_NO_6x6mm_H9.5mm, symbol Switch:SW_MEC_5E
- added SW6: BUTTON4, Button_Switch_SMD:SW_Push_1P1T_NO_6x6mm_H9.5mm, symbol Switch:SW_MEC_5E
- C82: value 100n -> 10n
- R127, R131: value 30k -> 33k
- R60: value 100k -> 10k; footprint (none) -> Resistor_SMD:R_0603_1608Metric
- R61: value 30k -> 10k; footprint (none) -> Resistor_SMD:R_0603_1608Metric
Connections:
- net +3V3: now also R60.1, R61.1, R102.1, R58.1
- net AREF_-10V: no longer R60.2
- net GND: now also C33.2, C34.2, C35.2, C36.2, SW3.1, SW3.2, SW4.1, SW4.2, SW5.1, SW5.2, SW6.1, SW6.2; no longer U12.12 (+)
- net AREF_3V0 renamed AREF_3V3
- net AREF_3V3: now also U12.13 (-); no longer R61.1
- new net +3.3VA: U12.12 (+)
- new net BUTTON1: C33.1, R58.2, SW3.3 (K), SW3.4 (A)
- new net BUTTON2: C34.1, R60.2, SW4.3 (K), SW4.4 (A)
- new net BUTTON3: C35.1, R61.2, SW5.3 (K), SW5.4 (A)
- new net BUTTON4: C36.1, R102.2, SW6.3 (K), SW6.4 (A)
Other:
- note added: "0…3.3V to -5.25…5.25V"
- note added: "SOFT BUTTONS"
- note added: "TODO: re-check levels"
- note added: "need separate 3v3 reference since\nVDDA not broken out on LCtech board"
- note added: "unity gain buffer"
- note removed: "0…3V to -5.25…5.25V"

Commit message: create README.md
Parts:
- R128, R132: value 105k -> 102k
Other:
- note added: "0…3.3V to -5.1…5.1V"
- note added: "need separate 3v3 reference since\nVDDA on LCtech board not available"
- note removed: "0…3.3V to -5.25…5.25V"
- note removed: "TODO: re-check levels"
- note removed: "need separate 3v3 reference since\nVDDA not broken out on LCtech board"
- moved on the sheet: C33, C34, C35, C36, R102, R58, R60, R61, SW3, SW4, SW5, SW6

Commit message: cleanup
Parts:
- removed C81: 1u, symbol Device:C_Small
- removed C82: 10n, symbol Device:C_Small
- removed U12: TL074, symbol Amplifier_Operational:TL074
- removed U20: TL072, symbol Amplifier_Operational:TL072
- added U12: TL072, symbol Amplifier_Operational:TL072
- added unit 2 of U19
- R62, R66: value 1.2k -> 1k
Connections:
- net GATE_OUT1: now also U12.3 (+)
- net GATE_OUT2: now also U12.5 (+)
- net GND: now also U19.5 (+)
- net VCC: now also U12.8 (V+)
- net VEE: now also U12.4 (V-)
- net at R104.1, R66.2, R68.2: now also U12.7
- net at R103.1, R62.2, R64.2: now also U12.1
- net at R63.1, R64.1: now also U12.2 (-)
- net at R67.1, R68.1: now also U12.6 (-)
- net at R133.1: now also U19.7
- net at C91.2, R130.1, R131.1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: now also U19.6 (-)
Other:
- note added: "VOLTAGE REFERENCE"
- note removed: "VOLTAGE REFERENCES"
- note removed: "need separate 3v3 reference since\nVDDA on LCtech board not available"
- note removed: "unity gain buffer"
- note removed: "unused"
- moved on the sheet: C33, C34, C35, C36, C63, C64, C88, C89, R102, R58, R60, R61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
