File: kicad/axoloti_429_eurorack/power.sch (KiCad schematic (older format))
At the start: 23 parts, among them J2 EURO_POWER, U3 MP1469, U4 LM1117-3.3, U5 LM1117-3.3

Commit message: cleanup
Parts:
- removed C28, C29: 47u, Capacitor_SMD:CP_Elec_4x5.4, symbol Device:CP1_Small
- removed C31: 100n, Capacitor_SMD:C_0603_1608Metric, symbol Device:C_Small
- removed R25: 4.7, Resistor_SMD:R_0603_1608Metric, symbol Device:R
- removed U4: LM1117-3.3, Package_TO_SOT_SMD:SOT-223-3_TabPin2, symbol Regulator_Linear:LM1117-3.3
Other:
- moved on the sheet: C30, C32, U5
Changed lines of the file:
@@
 Comment4 ""
 $EndDescr
-$Comp
-L power:+3.3V #PWR023
-U 1 1 5ECDF67F
-P 10275 2650
-AR Path="/5ECDA234/5ECDF67F" Ref="#PWR023"  Part="1"
-AR Path="/5ED86ED4/5ECDF67F" Ref="#PWR029"  Part="1"
-F 0 "#PWR029" H 10275 2500 50  0001 C CNN
-F 1 "+3.3V" H 10275 2800 50  0000 C CNN
-F 2 "" H 10275 2650 50  0001 C CNN
-F 3 "" H 10275 2650 50  0001 C CNN
-	1    10275 2650
-	1    0    0    -1
-$EndComp
-Wire Wire Line
-	8200 2800 8200 2650
-$Comp
-L Device:R R25
-U 1 1 5EDA1E36
-P 8475 2800
-F 0 "R25" V 8375 2800 50  0000 C CNN
-F 1 "4.7" V 8475 2800 50  0000 C CNN
-F 2 "Resistor_SMD:R_0603_1608Metric" V 8405 2800 50  0001 C CNN
-F 3 "" H 8475 2800 50  0001 C CNN
-	1    8475 2800
-	0    1    1    0
-$EndComp
-$Comp
-L Device:CP1_Small C28
-U 1 1 5EDA2BEA
-P 8775 2950
-F 0 "C28" H 8866 2996 50  0000 L CNN
-F 1 "47u" H 8866 2905 50  0000 L CNN
-F 2 "Capacitor_SMD:CP_Elec_4x5.4" H 8775 2950 50  0001 C CNN
-F 3 "" H 8775 2950 50  0001 C CNN
-	1    8775 2950
-	1    0    0    -1
-$EndComp
-Wire Wire Line
-	8625 2800 8775 2800
-Wire Wire Line
-	8775 2800 8775 2850
-Wire Wire Line
-	8775 2800 9075 2800
-Connection ~ 8775 2800
-Wire Wire Line
-	8775 3300 9375 3300
-$Comp
-L Device:C_Small C31
-U 1 1 5EDADB63
-P 10275 2900
-F 0 "C31" H 10367 2946 50  0000 L CNN
-F 1 "100n" H 10367 2855 50  0000 L CNN
-F 2 "Capacitor_SMD:C_0603_1608Metric" H 10275 2900 50  0001 C CNN
-F 3 "" H 10275 2900 50  0001 C CNN
-	1    10275 2900
-	1    0    0    -1
-$EndComp
-Wire Wire Line
-	9375 3300 9975 3300
-Wire Wire Line
-	9975 3300 9975 3000
-Connection ~ 9375 3300
-Wire Wire Line
-	9975 3300 10275 3300
-Wire Wire Line
-	10275 3300 10275 3000
-Connection ~ 9975 3300
-Wire Wire Line
-	10275 2650 10275 2800
-Connection ~ 10275 2800
-Wire Wire Line
-	8900 4075 9075 4075
+Wire Wire Line
+	8725 3175 8900 3175
 $Comp
 L Device:CP1_Small C30
 U 1 1 5EDBC007
-P 9975 4175
-F 0 "C30" H 10066 4221 50  0000 L CNN
-F 1 "47u" H 10066 4130 50  0000 L CNN
-F 2 "Capacitor_SMD:CP_Elec_4x5.4" H 9975 4175 50  0001 C CNN
-F 3 "" H 9975 4175 50  0001 C CNN
-	1    9975 4175
+P 9800 3275
+F 0 "C30" H 9891 3321 50  0000 L CNN
+F 1 "47u" H 9891 3230 50  0000 L CNN
+F 2 "Capacitor_SMD:CP_Elec_4x5.4" H 9800 3275 50  0001 C CNN
+F 3 "" H 9800 3275 50  0001 C CNN
+	1    9800 3275
 	1    0    0    -1
 $EndComp
@@
 L Device:C_Small C32
 U 1 1 5EDBC00E
-P 10275 4175
-F 0 "C32" H 10367 4221 50  0000 L CNN
-F 1 "100n" H 10367 4130 50  0000 L CNN
-F 2 "Capacitor_SMD:C_0603_1608Metric" H 10275 4175 50  0001 C CNN
-F 3 "" H 10275 4175 50  0001 C CNN
-	1    10275 4175
-	1    0    0    -1
-$EndComp
-Wire Wire Line
-	9975 4075 10275 4075
-Connection ~ 9975 4075
-Wire Wire Line
-	9375 4575 9975 4575
-Wire Wire Line
-	9975 4575 9975 4275
-Wire Wire Line
-	9975 4575 10275 4575
-Wire Wire Line
-	10275 4575 10275 4275
-Connection ~ 9975 4575
-Wire Wire Line
-	10275 3975 10275 4075
-Connection ~ 10275 4075
-Connection ~ 9975 2800
-Wire Wire Line
-	9975 2800 10275 2800
-$Comp
-L Device:CP1_Small C29
-U 1 1 5EDA7B97
-P 9975 2900
-F 0 "C29" H 10066 2946 50  0000 L CNN
-F 1 "47u" H 10066 2855 50  0000 L CNN
-F 2 "Capacitor_SMD:CP_Elec_4x5.4" H 9975 2900 50  0001 C CNN
-F 3 "" H 9975 2900 50  0001 C CNN
-	1    9975 2900
-	1    0    0    -1
-$EndComp
+P 10100 3275
+F 0 "C32" H 10192 3321 50  0000 L CNN
+F 1 "100n" H 10192 3230 50  0000 L CNN
+F 2 "Capacitor_SMD:C_0603_1608Metric" H 10100 3275 50  0001 C CNN
+F 3 "" H 10100 3275 50  0001 C CNN
+	1    10100 3275
+	1    0    0    -1
+$EndComp
+Wire Wire Line
+	9800 3175 10100 3175
+Connection ~ 9800 3175
+Wire Wire Line
+	9200 3675 9800 3675
+Wire Wire Line
+	9800 3675 9800 3375
+Wire Wire Line
+	9800 3675 10100 3675
+Wire Wire Line
+	10100 3675 10100 3375
+Connection ~ 9800 3675
+Wire Wire Line
+	10100 3075 10100 3175
+Connection ~ 10100 3175
 $Comp
 L power:+3.3VA #PWR0106
 U 1 1 60F2698F
-P 10275 3975
-F 0 "#PWR0106" H 10275 3825 50  0001 C CNN
-F 1 "+3.3VA" H 10290 4148 50  0000 C CNN
-F 2 "" H 10275 3975 50  0001 C CNN
-F 3 "" H 10275 3975 50  0001 C CNN
-	1    10275 3975
-	1    0    0    -1
-$EndComp
-$Comp
-L Regulator_Linear:LM1117-3.3 U4
-U 1 1 60F2FA3D
-P 9375 2800
-F 0 "U4" H 9375 3042 50  0000 C CNN
-F 1 "LM1117-3.3" H 9375 2951 50  0000 C CNN
-F 2 "Package_TO_SOT_SMD:SOT-223-3_TabPin2" H 9375 2800 50  0001 C CNN
-F 3 "http://www.ti.com/lit/ds/symlink/lm1117.pdf" H 9375 2800 50  0001 C CNN
-	1    9375 2800
+P 10100 3075
+F 0 "#PWR0106" H 10100 2925 50  0001 C CNN
+F 1 "+3.3VA" H 10115 3248 50  0000 C CNN
+F 2 "" H 10100 3075 50  0001 C CNN
+F 3 "" H 10100 3075 50  0001 C CNN
+	1    10100 3075
 	1    0    0    -1
 $EndComp
@@
 L Regulator_Linear:LM1117-3.3 U5
 U 1 1 60F3161A
-P 9375 4075
-F 0 "U5" H 9375 4317 50  0000 C CNN
-F 1 "LM1117-3.3" H 9375 4226 50  0000 C CNN
-F 2 "Package_TO_SOT_SMD:SOT-223-3_TabPin2" H 9375 4075 50  0001 C CNN
-F 3 "http://www.ti.com/lit/ds/symlink/lm1117.pdf" H 9375 4075 50  0001 C CNN
-	1    9375 4075
-	1    0    0    -1
-$EndComp
-Wire Wire Line
-	9375 3100 9375 3300
-Wire Wire Line
-	9675 2800 9975 2800
-Wire Wire Line
-	9375 4375 9375 4575
-Wire Wire Line
-	9675 4075 9975 4075
+P 9200 3175
+F 0 "U5" H 9200 3417 50  0000 C CNN
+F 1 "LM1117-3.3" H 9200 3326 50  0000 C CNN
+F 2 "Package_TO_SOT_SMD:SOT-223-3_TabPin2" H 9200 3175 50  0001 C CNN
+F 3 "http://www.ti.com/lit/ds/symlink/lm1117.pdf" H 9200 3175 50  0001 C CNN
+	1    9200 3175
+	1    0    0    -1
+$EndComp
+Wire Wire Line
+	9200 3475 9200 3675
+Wire Wire Line
+	9500 3175 9800 3175
 $Comp
 L Connector_Generic:Conn_02x05_Odd_Even J2
@@
 	2875 3375 2575 3375
 Connection ~ 2575 3375
-Wire Wire Line
-	8775 3050 8775 3300
-$Comp
-L power:VCC #PWR073
-U 1 1 615B1F7F
-P 8200 2650
-F 0 "#PWR073" H 8200 2500 50  0001 C CNN
-F 1 "VCC" H 8215 2823 50  0000 C CNN
-F 2 "" H 8200 2650 50  0001 C CNN
-F 3 "" H 8200 2650 50  0001 C CNN
-	1    8200 2650
-	1    0    0    -1
-$EndComp
-$Comp
-L power:GND #PWR075
-U 1 1 615B3B90
-P 9375 3375
-F 0 "#PWR075" H 9375 3125 50  0001 C CNN
-F 1 "GND" H 9380 3202 50  0000 C CNN
-F 2 "" H 9375 3375 50  0001 C CNN
-F 3 "" H 9375 3375 50  0001 C CNN
-	1    9375 3375
-	1    0    0    -1
-$EndComp
-Wire Wire Line
-	9375 3375 9375 3300
-Wire Wire Line
-	8200 2800 8325 2800
 $Comp
 L power:VCC #PWR074
 U 1 1 615B5E5E
-P 8900 3975
-F 0 "#PWR074" H 8900 3825 50  0001 C CNN
-F 1 "VCC" H 8915 4148 50  0000 C CNN
-F 2 "" H 8900 3975 50  0001 C CNN
-F 3 "" H 8900 3975 50  0001 C CNN
-	1    8900 3975
-	1    0    0    -1
-$EndComp
-Wire Wire Line
-	8900 3975 8900 4075
+P 8725 3075
+F 0 "#PWR074" H 8725 2925 50  0001 C CNN
+F 1 "VCC" H 8740 3248 50  0000 C CNN
+F 2 "" H 8725 3075 50  0001 C CNN
+F 3 "" H 8725 3075 50  0001 C CNN
+	1    8725 3075
+	1    0    0    -1
+$EndComp
+Wire Wire Line
+	8725 3075 8725 3175
 $Comp
 L TT-rescue:MP1469 U3
@@
 L power:GNDA #PWR091
 U 1 1 611A99CC
-P 9375 4575
-F 0 "#PWR091" H 9375 4325 50  0001 C CNN
-F 1 "GNDA" H 9380 4402 50  0000 C CNN
-F 2 "" H 9375 4575 50  0001 C CNN
-F 3 "" H 9375 4575 50  0001 C CNN
-	1    9375 4575
-	1    0    0    -1
-$EndComp
-Connection ~ 9375 4575
+P 9200 3675
+F 0 "#PWR091" H 9200 3425 50  0001 C CNN
+F 1 "GNDA" H 9205 3502 50  0000 C CNN
+F 2 "" H 9200 3675 50  0001 C CNN
+F 3 "" H 9200 3675 50  0001 C CNN
+	1    9200 3675
+	1    0    0    -1
+$EndComp
+Connection ~ 9200 3675
 Text Notes 5600 1475 0    79   ~ 0
 POWER
