File: kicad/axoloti_429_eurorack/usb.sch (KiCad schematic (older format))
At the start: 12 parts, among them J12 USB_A, J13 USB_B, U16 USBLC6-2P6, U21 STMPS2141, U9 USBLC6-2P6

Commit message: cleanup
Parts:
- J12: value USB_A -> USB_A_VERTICAL
- J13: value USB_B -> USB_MICRO_B_VERTICAL; footprint (none) -> Connector_USB:USB_Micro-B_Wuerth_614105150721_Vertical
Other:
- note added: "TODO\nstill don't understand VBUS"
Changed lines of the file:
@@
 P 6750 4150
 F 0 "J12" H 6807 4617 50  0000 C CNN
-F 1 "USB_A" H 6807 4526 50  0000 C CNN
+F 1 "USB_A_VERTICAL" H 6807 4526 50  0000 C CNN
 F 2 "w_connector:MOLEX_USB_105057" H 6900 4100 50  0001 C CNN
 F 3 " ~" H 6900 4100 50  0001 C CNN
@@
 P 2350 3250
 F 0 "J13" H 2407 3717 50  0000 C CNN
-F 1 "USB_B" H 2407 3626 50  0000 C CNN
-F 2 "" H 2500 3200 50  0001 C CNN
+F 1 "USB_MICRO_B_VERTICAL" H 2407 3626 50  0000 C CNN
+F 2 "Connector_USB:USB_Micro-B_Wuerth_614105150721_Vertical" H 2500 3200 50  0001 C CNN
 F 3 " ~" H 2500 3200 50  0001 C CNN
 	1    2350 3250
@@
 Wire Wire Line
 	7550 3950 7250 3950
+Text Notes 4525 2600 0    50   ~ 0
+TODO\nstill don't understand VBUS
 $EndSCHEMATC
